Commit message: Add inertia and reduce the meshes

File: k3_test_description/urdf/robot_k3_test.urdf.xacro (robot description, xacro)
@@ -44,7 +44,7 @@
             </collision>
             <inertial>
-                <origin xyz="0 0 0" rpy="0 0 ${dir * 90*pi/180}"/>
+                <origin xyz="-0.005351 0 0" rpy="0 0 ${dir * 90*pi/180}"/>
                 <mass value="1.0"/>
-                <inertia ixx="1.0" ixy="0.0" ixz="0.0" iyy="1.0" iyz="0.0" izz="1.0"/>
+                <inertia ixx="0.000051226" ixy="0.0" ixz="0.0" iyy="0.001861631" iyz="0.0" izz="0.001859351"/>
             </inertial>
         </link>
@@ -69,6 +69,6 @@
             <inertial>
                 <origin xyz="0 0 0" rpy="0 0 ${dir * 90*pi/180}"/>
-                <mass value="5.0"/>
-                <inertia ixx="1.0" ixy="0.0" ixz="0.0" iyy="1.0" iyz="0.0" izz="1.0"/>
+                <mass value="12.0"/>
+                <inertia ixx="0.037394" ixy="0.0" ixz="0.0" iyy="0.024470" iyz="0.0" izz="0.024470"/>
             </inertial>
         </link>
@@ -98,7 +98,7 @@
             </collision>
             <inertial>
-                <origin xyz="0 0 0" rpy="0 0 0"/>
-                <mass value="1.0"/>
-                <inertia ixx="1.0" ixy="0.0" ixz="0.0" iyy="1.0" iyz="0.0" izz="1.0"/>
+                <origin xyz="0 0 -0.01" rpy="0 0 0"/>
+                <mass value="1.579"/>
+                <inertia ixx="0.00133437338" ixy="0.0" ixz="0.0" iyy="0.00133595613" iyz="0.0" izz="0.00254792224"/>
             </inertial>
         </link>
@@ -122,7 +122,7 @@
             </collision>
             <inertial>
-                <origin xyz="0 0 0" rpy="0 0 0"/>
-                <mass value="1.0"/>
-                <inertia ixx="1.0" ixy="0.0" ixz="0.0" iyy="1.0" iyz="0.0" izz="1.0"/>
+                <origin xyz="-0.006856 0 -0.022825" rpy="0 0 0"/>
+                <mass value="1.824"/>
+                <inertia ixx="0.00162071448" ixy="0.0" ixz="0.0" iyy="0.00210140087" iyz="0.0" izz="0.00205468149"/>
             </inertial>
         </link>
@@ -148,6 +148,6 @@
             <inertial>
                 <origin xyz="0 0 0" rpy="0 0 0"/>
-                <mass value="1.0"/>
-                <inertia ixx="1.0" ixy="0.0" ixz="0.0" iyy="1.0" iyz="0.0" izz="1.0"/>
+                <mass value="0.319"/>
+                <inertia ixx="0.00039368351" ixy="0.0" ixz="0.0" iyy="0.00002810787" iyz="0.0" izz="0.00038530588"/>
             </inertial>
         </link>
@@ -167,15 +167,13 @@
             </visual>
             <collision>
-                <origin xyz="0 0 0" rpy="${90*pi/180} 0 0"/>
-                <geometry>
-                    <!-- <mesh filename="package://k3_test_description/meshes/caster_wheel.dae" scale="1 1 1"/> -->
-                    <cylinder radius="0.0375" length="0.030"/>
-                </geometry>
-            </collision>
-            <inertial>
-                <origin xyz="0 0 0" rpy="${90*pi/180} 0 0"/>
-                <mass value="1.0"/>
-                <!-- <inertia ixx="1.0" ixy="0.0" ixz="0.0" iyy="1.0" iyz="0.0" izz="1.0"/> -->
-                    <xacro:cylinder_inertia m="1.0" r="0.0375" h="0.030"/>
+                <origin xyz="0 0 0" rpy="0 0 ${90*pi/180}"/>
+                <geometry>
+                    <mesh filename="package://k3_test_description/meshes/caster_wheel.dae" scale="1 1 1"/>
+                </geometry>
+            </collision>
+            <inertial>
+                <origin xyz="0 0 0" rpy="0 0 ${90*pi/180}"/>
+                <mass value="0.936"/>
+                <inertia ixx="0.00065654885" ixy="0.0" ixz="0.0" iyy="0.00039382798" iyz="0.0" izz="0.00039372956"/>
             </inertial>
         </link>
@@ -201,6 +199,6 @@
             <inertial>
                 <origin xyz="0 0 0" rpy="0 0 ${-90*pi/180}"/>
-                <mass value="1.0"/>
-                <inertia ixx="1.0" ixy="0.0" ixz="0.0" iyy="1.0" iyz="0.0" izz="1.0"/>
+                <mass value="0.936"/>
+                <inertia ixx="0.00065654885" ixy="0.0" ixz="0.0" iyy="0.00039382798" iyz="0.0" izz="0.00039372956"/>
             </inertial>
         </link>
