Commit message: Add map for testing

File: k3_test_description/urdf/rack_900.urdf.xacro (robot description, xacro)
@@ -1,5 +1,6 @@
 <?xml version="1.0"?>
 <robot name="rack_900" xmlns:xacro="http://www.ros.org/wiki/xacro">
-    <link name="rack_boxy">
+    <link name="rack_base_link"/>
+    <link name="rack_box">
         <visual>
             <origin xyz="0 0 0" rpy="0 0 0"/>
@@ -15,8 +16,16 @@
         </collision>
         <inertial>
-            <origin xyz="0 0 2.160" rpy="0 0 0"/>
+            <origin xyz="0 0 1.160" rpy="0 0 0"/>
             <mass value="100"/>
             <inertia ixx="54.91434330682" ixy="0.0" ixz="0.0" iyy="54.91434330682" iyz="0.0" izz="22.4138576779"/>
         </inertial>
     </link>
+    <joint name="rack_base_link_fixed" type="fixed">
+        <parent link="rack_base_link"/>
+        <child link="rack_box"/>
+        <origin xyz="0 0 0" rpy="0 0 0"/>
+    </joint>
+    <gazebo reference="rack_base_link">
+        <gravity>0</gravity>
+    </gazebo>
 </robot>

File: k3_test_description/urdf/robot_k3_test.urdf.xacro (robot description, xacro)
@@ -271,5 +271,5 @@
         <axis xyz="0 0 1"/>
         <origin xyz="0 0 0.1555" rpy="0 0 0"/>
-        <limit effort="100" velocity="0.2" lower="0" upper="0.04"/>
+        <limit effort="1000" velocity="0.05" lower="0" upper="0.045"/>
     </joint>
     <xacro:insert_position_transmission name="top_lift_joint"/>
